File: GlasgowICAdapter/GlasgowICAdapter.kicad_sch (KiCad schematic)
At the start: 19 parts, among them J1 PORT A, J10 PORT A IO, J11 PORT B IO, J2 PORT B, J3 ZIF_SOCKET, J4 EN_U1, J5 EN_U2, J6 ZIF_IO_LEFT, J7 EN_U3, J8 EN_U4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

Commit message: Added proper footprints to all symbols
Parts:
- J1, J2: footprint SFH11-PBPC-D10-ST-BK:SULLINS_SFH11-PBPC-D10-ST-BK -> SFH11_PBPC_D10_ST_BK:CONN_SFH11-PBPC-D10-ST-BK_SUL
- J10, J11: footprint (none) -> Connector_PinHeader_2.54mm:PinHeader_2x10_P2.54mm_Vertical
- J3: footprint (none) -> Socket:DIP_Socket-32_W11.9mm_W12.7mm_W15.24mm_W17.78mm_W18.5mm_3M_232-1285-00-0602J
- J4, J5, J7, J8: footprint (none) -> Connector_PinHeader_2.54mm:PinHeader_1x02_P2.54mm_Vertical
- J6, J9: footprint (none) -> Connector_PinHeader_2.54mm:PinHeader_1x16_P2.54mm_Vertical
- R1, R2, R3, R4: footprint (none) -> Resistor_THT:R_Axial_DIN0204_L3.6mm_D1.6mm_P7.62mm_Horizontal
- U1, U2, U4, U5: footprint RSV0016A -> TMUX1029RSVR:RSV0016A
Changed lines of the file:
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@@
 			)
 		)
-		(property "Footprint" "RSV0016A"
+		(property "Footprint" "TMUX1029RSVR:RSV0016A"
 			(at 157.48 49.53 0)
 			(effects
@@
 			)
 		)
-		(property "Footprint" ""
+		(property "Footprint" "Connector_PinHeader_2.54mm:PinHeader_1x02_P2.54mm_Vertical"
 			(at 260.35 29.21 0)
 			(effects
@@
 			)
 		)
-		(property "Footprint" ""
+		(property "Footprint" "Resistor_THT:R_Axial_DIN0204_L3.6mm_D1.6mm_P7.62mm_Horizontal"
 			(at 182.118 24.13 90)
 			(effects
@@
 			)
 		)
-		(property "Footprint" ""
+		(property "Footprint" "Connector_PinHeader_2.54mm:PinHeader_1x02_P2.54mm_Vertical"
 			(at 187.96 87.63 0)
 			(effects
@@
 			)
 		)
-		(property "Footprint" ""
+		(property "Footprint" "Connector_PinHeader_2.54mm:PinHeader_2x10_P2.54mm_Vertical"
 			(at 86.36 36.83 0)
 			(effects
@@
 			)
 		)
-		(property "Footprint" "RSV0016A"
+		(property "Footprint" "TMUX1029RSVR:RSV0016A"
 			(at 229.87 107.95 0)
 			(effects
@@
 			)
 		)
-		(property "Footprint" ""
+		(property "Footprint" "Connector_PinHeader_2.54mm:PinHeader_1x16_P2.54mm_Vertical"
 			(at 77.47 114.3 0)
 			(effects
@@
 			)
 		)
-		(property "Footprint" ""
+		(property "Footprint" "Resistor_THT:R_Axial_DIN0204_L3.6mm_D1.6mm_P7.62mm_Horizontal"
 			(at 254.508 24.13 90)
 			(effects
@@
 			)
 		)
-		(property "Footprint" ""
+		(property "Footprint" "Connector_PinHeader_2.54mm:PinHeader_1x16_P2.54mm_Vertical"
 			(at 80.01 116.84 0)
 			(effects
@@
 			)
 		)
-		(property "Footprint" "RSV0016A"
+		(property "Footprint" "TMUX1029RSVR:RSV0016A"
 			(at 229.87 49.53 0)
 			(effects
@@
 			)
 		)
-		(property "Footprint" ""
+		(property "Footprint" "Resistor_THT:R_Axial_DIN0204_L3.6mm_D1.6mm_P7.62mm_Horizontal"
 			(at 254.508 82.55 90)
 			(effects
@@
 			)
 		)
-		(property "Footprint" ""
+		(property "Footprint" "Socket:DIP_Socket-32_W11.9mm_W12.7mm_W15.24mm_W17.78mm_W18.5mm_3M_232-1285-00-0602J"
 			(at 40.64 114.3 0)
 			(effects
@@
 			)
 		)
-		(property "Footprint" "RSV0016A"
+		(property "Footprint" "TMUX1029RSVR:RSV0016A"
 			(at 157.48 107.95 0)
 			(effects
@@
 			)
 		)
-		(property "Footprint" ""
+		(property "Footprint" "Connector_PinHeader_2.54mm:PinHeader_1x02_P2.54mm_Vertical"
 			(at 260.35 87.63 0)
 			(effects
@@
 			)
 		)
-		(property "Footprint" ""
+		(property "Footprint" "Connector_PinHeader_2.54mm:PinHeader_2x10_P2.54mm_Vertical"
 			(at 86.36 72.39 0)
 			(effects
@@
 			)
 		)
-		(property "Footprint" ""
+		(property "Footprint" "Connector_PinHeader_2.54mm:PinHeader_1x02_P2.54mm_Vertical"
 			(at 187.96 29.21 0)
 			(effects
@@
 			)
 		)
-		(property "Footprint" "SFH11-PBPC-D10-ST-BK:SULLINS_SFH11-PBPC-D10-ST-BK"
+		(property "Footprint" "SFH11_PBPC_D10_ST_BK:CONN_SFH11-PBPC-D10-ST-BK_SUL"
 			(at 41.91 72.39 0)
 			(effects
@@
 			)
 		)
-		(property "Footprint" "SFH11-PBPC-D10-ST-BK:SULLINS_SFH11-PBPC-D10-ST-BK"
+		(property "Footprint" "SFH11_PBPC_D10_ST_BK:CONN_SFH11-PBPC-D10-ST-BK_SUL"
 			(at 41.91 36.83 0)
 			(effects
@@
 			)
 		)
-		(property "Footprint" ""
+		(property "Footprint" "Resistor_THT:R_Axial_DIN0204_L3.6mm_D1.6mm_P7.62mm_Horizontal"
 			(at 182.118 82.55 90)
 			(effects

Commit message: Slightly imporved schematic
Parts:
- J10, J11: symbol Connector_Generic:Conn_02x10_Counter_Clockwise -> Connector_Generic:Conn_02x10_Odd_Even
Connections:
- net GND: now also J10.20 (Pin_20), J10.4 (Pin_4), J10.6 (Pin_6), J10.8 (Pin_8), J11.11 (Pin_11), J11.13 (Pin_13), J11.15 (Pin_15), J11.17 (Pin_17); no longer J10.11 (Pin_11), J10.13 (Pin_13), J10.15 (Pin_15), J10.17 (Pin_17), J11.20 (Pin_20), J11.4 (Pin_4), J11.6 (Pin_6), J11.8 (Pin_8), U1.1 (NC), U2.1 (NC), U4.1 (NC), U5.1 (NC)
- net PA0: now also J10.3 (Pin_3); no longer J10.2 (Pin_2)
- net PA1: now also J10.5 (Pin_5); no longer J10.3 (Pin_3)
- net PA2: now also J10.7 (Pin_7); no longer J10.4 (Pin_4)
- net PA3: now also J10.9 (Pin_9); no longer J10.5 (Pin_5)
- net PA4: now also J10.11 (Pin_11); no longer J10.6 (Pin_6)
- net PA5: now also J10.13 (Pin_13); no longer J10.7 (Pin_7)
- net PA6: now also J10.15 (Pin_15); no longer J10.8 (Pin_8)
- net PA7: now also J10.17 (Pin_17); no longer J10.9 (Pin_9)
- net PB0: now also J11.18 (Pin_18); no longer J11.12 (Pin_12)
- net PB1: now also J11.16 (Pin_16); no longer J11.13 (Pin_13)
- net PB3: now also J11.12 (Pin_12); no longer J11.15 (Pin_15)
- net PB4: now also J11.10 (Pin_10); no longer J11.16 (Pin_16)
- net PB5: now also J11.8 (Pin_8); no longer J11.17 (Pin_17)
- net PB6: now also J11.6 (Pin_6); no longer J11.18 (Pin_18)
- net PB7: now also J11.4 (Pin_4); no longer J11.19 (Pin_19)
- net VB SENSE: now also J11.20 (Pin_20); no longer J11.11 (Pin_11)
- net VIOA: now also J10.2 (Pin_2); no longer J10.20 (Pin_20)
- net VIOB: now also J11.19 (Pin_19); no longer J11.10 (Pin_10)
Changed lines of the file:
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@@
 	(paper "A4")
 	(junction
-		(at 135.89 87.63)
-		(diameter 0)
-		(color 0 0 0 0)
-	)
-	(junction
 		(at 57.15 31.75)
 		(diameter 0)
@@
 	)
 	(junction
-		(at 208.28 87.63)
-		(diameter 0)
-		(color 0 0 0 0)
-	)
-	(junction
 		(at 78.74 64.77)
 		(diameter 0)
@@
 	)
 	(junction
-		(at 208.28 29.21)
-		(diameter 0)
-		(color 0 0 0 0)
-	)
-	(junction
-		(at 135.89 29.21)
-		(diameter 0)
-		(color 0 0 0 0)
-	)
-	(junction
 		(at 26.67 67.31)
 		(diameter 0)
@@
 	(wire
 		(pts
-			(xy 135.89 29.21) (xy 137.16 29.21)
-		)
-		(stroke
-			(width 0)
-			(type default)
-		)
-	)
-	(wire
-		(pts
 			(xy 93.98 82.55) (xy 96.52 82.55)
 		)
@@
 	(wire
 		(pts
-			(xy 135.89 97.79) (xy 137.16 97.79)
-		)
-		(stroke
-			(width 0)
-			(type default)
-		)
-	)
-	(wire
-		(pts
 			(xy 69.85 132.08) (xy 72.39 132.08)
 		)
@@
 	(wire
 		(pts
-			(xy 208.28 87.63) (xy 208.28 97.79)
-		)
-		(stroke
-			(width 0)
-			(type default)
-		)
-	)
-	(wire
-		(pts
 			(xy 85.09 96.52) (xy 87.63 96.52)
 		)
@@
 	(wire
 		(pts
-			(xy 208.28 87.63) (xy 209.55 87.63)
-		)
-		(stroke
-			(width 0)
-			(type default)
-		)
-	)
-	(wire
-		(pts
 			(xy 26.67 72.39) (xy 29.21 72.39)
 		)
@@
 	(wire
 		(pts
-			(xy 208.28 97.79) (xy 209.55 97.79)
-		)
-		(stroke
-			(width 0)
-			(type default)
-		)
-	)
-	(wire
-		(pts
-			(xy 208.28 29.21) (xy 209.55 29.21)
-		)
-		(stroke
-			(width 0)
-			(type default)
-		)
-	)
-	(wire
-		(pts
 			(xy 78.74 31.75) (xy 81.28 31.75)
 		)
@@
 	(wire
 		(pts
-			(xy 135.89 29.21) (xy 135.89 39.37)
-		)
-		(stroke
-			(width 0)
-			(type default)
-		)
-	)
-	(wire
-		(pts
 			(xy 195.58 87.63) (xy 199.39 87.63)
 		)
@@
 	(wire
 		(pts
-			(xy 135.89 39.37) (xy 137.16 39.37)
-		)
-		(stroke
-			(width 0)
-			(type default)
-		)
-	)
-	(wire
-		(pts
 			(xy 78.74 44.45) (xy 81.28 44.45)
 		)
@@
 	(wire
 		(pts
-			(xy 199.39 29.21) (xy 208.28 29.21)
-		)
-		(stroke
-			(width 0)
-			(type default)
-		)
-	)
-	(wire
-		(pts
-			(xy 134.62 87.63) (xy 135.89 87.63)
+			(xy 199.39 29.21) (xy 209.55 29.21)
 		)
 		(stroke
@@
 	(wire
 		(pts
-			(xy 208.28 39.37) (xy 209.55 39.37)
-		)
-		(stroke
-			(width 0)
-			(type default)
-		)
-	)
-	(wire
-		(pts
 			(xy 85.09 129.54) (xy 87.63 129.54)
 		)
@@
 	(wire
 		(pts
-			(xy 134.62 29.21) (xy 135.89 29.21)
-		)
-		(stroke
-			(width 0)
-			(type default)
-		)
-	)
-	(wire
-		(pts
-			(xy 135.89 87.63) (xy 135.89 97.79)
+			(xy 134.62 29.21) (xy 137.16 29.21)
 		)
 		(stroke
@@
 	(wire
 		(pts
-			(xy 208.28 29.21) (xy 208.28 39.37)
-		)
-		(stroke
-			(width 0)
-			(type default)
-		)
-	)
-	(wire
-		(pts
 			(xy 78.74 67.31) (xy 78.74 64.77)
 		)
@@
 	(wire
 		(pts
-			(xy 135.89 87.63) (xy 137.16 87.63)
+			(xy 134.62 87.63) (xy 137.16 87.63)
 		)
 		(stroke
@@
 	(wire
 		(pts
-			(xy 199.39 87.63) (xy 208.28 87.63)
+			(xy 199.39 87.63) (xy 209.55 87.63)
 		)
 		(stroke
@@
 	)
 	(symbol
-		(lib_id "Connector_Generic:Conn_02x10_Counter_Clockwise")
+		(lib_id "Connector_Generic:Conn_02x10_Odd_Even")
 		(at 86.36 36.83 0)
 		(unit 1)
@@
 			)
 		)
-		(property "Description" "Generic connector, double row, 02x10, counter clockwise pin numbering scheme (similar to DIP package numbering), script generated (kicad-library-utils/schlib/autogen/connector/)"
+		(property "Description" "Generic connector, double row, 02x10, odd/even pin numbering scheme (row 1 odd numbers, row 2 even numbers), script generated (kicad-library-utils/schlib/autogen/connector/)"
 			(at 86.36 36.83 0)
 			(effects
@@
 	)
 	(symbol
-		(lib_id "Connector_Generic:Conn_02x10_Counter_Clockwise")
+		(lib_id "Connector_Generic:Conn_02x10_Odd_Even")
 		(at 86.36 72.39 0)
 		(unit 1)
@@
 			)
 		)
-		(property "Description" "Generic connector, double row, 02x10, counter clockwise pin numbering scheme (similar to DIP package numbering), script generated (kicad-library-utils/schlib/autogen/connector/)"
+		(property "Description" "Generic connector, double row, 02x10, odd/even pin numbering scheme (row 1 odd numbers, row 2 even numbers), script generated (kicad-library-utils/schlib/autogen/connector/)"
 			(at 86.36 72.39 0)
 			(effects
